Commit message: Add HRI experiment scripts and Unity integration
- Add EEG recording/analysis scripts (eeg_recorder, analyze_edf, analyze_xdf)
- Add Unity bridge and VR teleop support
- Add pick and place scripts for robot manipulation
- Add gripper test and robot dance demos
- Update configs for gripper and kinematics
- Update .gitignore for Python cache files

🤖 Generated with [Claude Code](https://claude.com/claude-code)

Co-Authored-By: Claude Opus 4.5 <noreply@anthropic.com>

File: annin_ar4_description/urdf/ar_gripper_macro.xacro (robot description, xacro)
@@ -75,5 +75,5 @@
       <child link="${tf_prefix}gripper_jaw1_link"/>
       <axis xyz="-1 0 0"/>
-      <limit lower="0" upper="0.014" effort="-1" velocity="1.0"/>
+      <limit lower="0" upper="0.020" effort="-1" velocity="1.0"/>
     </joint>
     <joint name="${tf_prefix}gripper_jaw2_joint" type="prismatic">
@@ -82,5 +82,5 @@
       <child link="${tf_prefix}gripper_jaw2_link"/>
       <axis xyz="-1 0 0"/>
-      <limit lower="0" upper="0.014" effort="1000" velocity="1.0"/>
+      <limit lower="0" upper="0.020" effort="1000" velocity="1.0"/>
       <mimic joint="${tf_prefix}gripper_jaw1_joint" multiplier="1" offset="0"/>
     </joint>
